File: pcb/LowJungle.kicad_pcb (KiCad board)
At the start: 2 copper layers, 3.6 x 3.3 mm, 255 parts

Commit message: Move all hot swap socket to flipping right side
Parts:
- CH1, CH10, CH12, CH13, CH14, CH15, CH16, CH18, CH19, CH2, CH20, CH21, CH22, CH24, CH25, CH26, CH27, CH28, CH29, CH30, CH31, CH32, CH33, CH34, CH35, CH36, CH37, CH38, CH39, CH40, CH41, CH42, CH43, CH44, CH45, CH46, CH47, CH48, CH49, CH50, CH51, CH52, CH53, CH54, CH55, CH56, CH57, CH58, CH59, CH60, CH61, CH62, CH63, CH64, CH65, CH67, CH7, CH74, CH75, CH76, CH77, CH78, CH79, CH8, CH80, CH81, CH82, CH83, CH84, CH85, CH9: footprint PCM_marbastlib-xp-gateron_lp:SW_KS33_HS_KS-2P02B01-02_HS_1u -> 0_Custom:SW_KS33_HS_KS-2P02B01-02_1u
- CH11, CH17, CH5, CH6, CH66, CH71, CH72, CH73: footprint PCM_marbastlib-xp-gateron_lp:SW_KS33_HS_KS-2P02B01-02_1.25u -> 0_Custom:SW_KS33_HS_KS-2P02B01-02_1.25u
- CH23: footprint PCM_marbastlib-xp-gateron_lp:SW_KS33_HS_KS-2P02B01-02_HS_1u -> 0_Custom:SW_KS33_HS_KS-2P02B01-02_6.25
- CH3: footprint PCM_marbastlib-xp-gateron_lp:SW_KS33_HS_KS-2P02B01-02_1.5u -> 0_Custom:SW_KS33_HS_KS-2P02B01-02_1.5u
- CH4: footprint PCM_marbastlib-xp-gateron_lp:SW_KS33_HS_KS-2P02B01-02_1.75u -> 0_Custom:SW_KS33_HS_KS-2P02B01-02_1.75u
- CH68: footprint PCM_marbastlib-xp-gateron_lp:SW_KS33_HS_KS-2P02B01-02_1.5u -> 0_Custom:SW_KS33_HS_KS-2P02B01-02_2u
- CH69: footprint PCM_marbastlib-xp-gateron_lp:SW_KS33_HS_KS-2P02B01-02_1.25u -> 0_Custom:SW_KS33_HS_KS-2P02B01-02_Enter
- CH70: footprint PCM_marbastlib-xp-gateron_lp:SW_KS33_HS_KS-2P02B01-02_HS_1u -> 0_Custom:SW_KS33_HS_KS-2P02B01-02_2.75u
- D16, LED1: moved to B.Cu
- moved D70 35.7 mm to (278.6, 116.2)
- moved D66 21.4 mm to (221.5, 135.3)
- moved D69 21.3 mm to (292.9, 87.6)
- moved D16 20.5 mm to (71.4, 123.8), turned to 90 degrees
- moved D18 19.1 mm to (85.7, 30.5)
- moved D43 19.1 mm to (171.4, 30.5)
- moved D48 19.1 mm to (190.5, 30.5)
- moved D58 19.1 mm to (238.1, 30.5)
- moved D67 19.1 mm to (257.2, 30.5)
- moved D75 19.1 mm to (295.3, 30.5)
- moved D1 19.1 mm to (28.6, 30.5)
- moved D12 19.1 mm to (66.7, 30.5)
- moved D24 19.1 mm to (104.8, 30.5)
- moved D29 19.1 mm to (123.8, 30.5)
- moved D38 19.1 mm to (152.4, 30.5)
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Other:
- board size 3.6 x 3.3 mm -> 378.6 x 152.4 mm

Commit message: Routing
Parts:
- D16: moved to F.Cu
- moved D16 7.62 mm to (71.4, 116.2), turned to -90 degrees
- moved D19 7.62 mm to (85.7, 59.1), turned to -90 degrees
Routing:
- net /KeyMatrix/COLUM_8: track 0.00 -> 306.4 mm, vias 0 -> 2
- net /KeyMatrix/COLUM_3: track 0.00 -> 223.5 mm, vias 0 -> 1
- net /KeyMatrix/COLUM_6: track 0.00 -> 209.6 mm
- net /KeyMatrix/COLUM_7: track 0.00 -> 203.3 mm
- net /KeyMatrix/COLUM_1: track 0.00 -> 197.3 mm, vias 0 -> 3
- net /KeyMatrix/COLUM_5: track 0.00 -> 195.5 mm
- net /KeyMatrix/COLUM_2: track 0.00 -> 189.4 mm
- net /KeyMatrix/COLUM_4: track 0.00 -> 185.4 mm
- net /KeyMatrix/COLUM_9: track 0.00 -> 119.6 mm, vias 0 -> 2
- net Net-(D62-A): track 0.00 -> 5.48 mm
- net Net-(D37-A): track 0.00 -> 5.48 mm
- net Net-(D54-A): track 0.00 -> 5.48 mm
- net Net-(D40-A): track 0.00 -> 5.48 mm
- net Net-(D43-A): track 0.00 -> 5.48 mm
- net Net-(D28-A): track 0.00 -> 5.48 mm
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
Commit message: ledsssssss
Parts:
- LED10, LED11, LED12, LED13, LED14, LED15, LED16, LED17, LED18, LED19, LED2, LED20, LED21, LED22, LED23, LED24, LED25, LED26, LED27, LED28, LED29, LED3, LED30, LED31, LED32, LED33, LED34, LED35, LED36, LED37, LED38, LED39, LED4, LED40, LED41, LED42, LED43, LED44, LED45, LED46, LED47, LED48, LED49, LED5, LED50, LED51, LED52, LED53, LED54, LED55, LED56, LED57, LED58, LED59, LED6, LED60, LED61, LED62, LED63, LED64, LED65, LED66, LED67, LED68, LED69, LED7, LED70, LED71, LED72, LED73, LED74, LED75, LED76, LED77, LED78, LED79, LED8, LED80, LED81, LED82, LED83, LED84, LED85, LED9: moved to B.Cu
- moved LED9 357.4 mm to (304.1, 32.9), turned to 180 degrees
- moved LED53 356.5 mm to (370.8, 80.5), turned to 180 degrees
- moved LED34 354.3 mm to (370.8, 61.5), turned to 180 degrees
- moved LED54 342.7 mm to (351.8, 80.5), turned to 180 degrees
- moved LED35 339.5 mm to (351.7, 61.5), turned to 180 degrees
- moved LED8 339.5 mm to (285.1, 33.0), turned to 180 degrees
- moved LED55 335.6 mm to (370.8, 137.8), turned to 180 degrees
- moved LED36 325.4 mm to (332.6, 61.5), turned to 180 degrees
- moved LED19 322.4 mm to (294.6, 61.5), turned to 180 degrees
- moved LED7 321.8 mm to (266.0, 33.0), turned to 180 degrees
- moved LED37 318.6 mm to (332.7, 80.5), turned to 180 degrees
- moved LED6 304.3 mm to (246.9, 33.0), turned to 180 degrees
- moved LED20 303.1 mm to (266.1, 61.5), turned to 180 degrees
- moved LED21 292.2 mm to (247.0, 61.5), turned to 180 degrees
- moved LED38 289.4 mm to (301.7, 90.0), turned to 180 degrees
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
Commit message: Added stabilizers
Parts:
- moved D68 8.33 mm to (277.4, 59.1)
- moved D70 8.33 mm to (270.3, 116.2)
Connections:
- LED1 pad 3: Net-(LED1-DIN) -> /LEDs/DIN
- LED18 pad 3: Net-(LED1-DOUT) -> Net-(LED18-DIN)
- LED2 pad 2: Net-(LED1-DIN) -> Net-(LED2-DOUT)
- LED2 pad 3: Net-(LED2-DIN) -> Net-(LED1-DOUT)
- LED3 pad 2: Net-(LED2-DIN) -> Net-(LED3-DOUT)
- LED3 pad 3: Net-(LED3-DIN) -> Net-(LED2-DOUT)
- LED4 pad 2: Net-(LED3-DIN) -> Net-(LED4-DOUT)
- LED4 pad 3: Net-(LED4-DIN) -> Net-(LED3-DOUT)
- LED5 pad 2: Net-(LED4-DIN) -> Net-(LED5-DOUT)
- LED5 pad 3: Net-(LED5-DIN) -> Net-(LED4-DOUT)
- LED55 pad 2: Net-(LED55-DOUT) -> unconnected-(LED55-DOUT-Pad2)
- LED56 pad 2: Net-(LED55-DIN) -> Net-(LED56-DOUT)
- LED6 pad 2: Net-(LED5-DIN) -> Net-(LED6-DOUT)
- LED6 pad 3: Net-(LED6-DIN) -> Net-(LED5-DOUT)
- LED7 pad 2: Net-(LED6-DIN) -> Net-(LED7-DOUT)
- LED7 pad 3: Net-(LED7-DIN) -> Net-(LED6-DOUT)
- LED72 pad 3: Net-(LED55-DOUT) -> Net-(LED56-DOUT)
- LED8 pad 2: Net-(LED7-DIN) -> Net-(LED8-DOUT)
- LED8 pad 3: Net-(LED8-DIN) -> Net-(LED7-DOUT)
- LED82 pad 2: unconnected-(LED82-DOUT-Pad2) -> Net-(LED55-DIN)
- LED9 pad 2: Net-(LED8-DIN) -> Net-(LED18-DIN)
- LED9 pad 3: /LEDs/DIN -> Net-(LED8-DOUT)
Routing:
- net Net-(D68-A): track 5.48 -> 15.3 mm
- net Net-(D70-A): track 5.48 -> 14.3 mm
- net /KeyMatrix/COLUM_7: track 203.3 -> 200.1 mm
Changed lines of the file:
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@@
 	(net 107 "Net-(LED1-DOUT)")
 	(net 108 "VBUS")
-	(net 109 "Net-(LED1-DIN)")
-	(net 110 "Net-(LED2-DIN)")
-	(net 111 "Net-(LED3-DIN)")
-	(net 112 "Net-(LED4-DIN)")
-	(net 113 "Net-(LED5-DIN)")
-	(net 114 "Net-(LED6-DIN)")
-	(net 115 "Net-(LED7-DIN)")
-	(net 116 "Net-(LED8-DIN)")
+	(net 109 "Net-(LED2-DOUT)")
+	(net 110 "Net-(LED3-DOUT)")
+	(net 111 "Net-(LED4-DOUT)")
+	(net 112 "Net-(LED5-DOUT)")
+	(net 113 "Net-(LED6-DOUT)")
+	(net 114 "Net-(LED7-DOUT)")
+	(net 115 "Net-(LED8-DOUT)")
+	(net 116 "Net-(LED18-DIN)")
 	(net 117 "/LEDs/DIN")
 	(net 118 "Net-(LED10-DOUT)")
@@
 	(net 161 "Net-(LED52-DIN)")
 	(net 162 "Net-(LED53-DIN)")
-	(net 163 "Net-(LED55-DOUT)")
+	(net 163 "unconnected-(LED55-DOUT-Pad2)")
 	(net 164 "Net-(LED55-DIN)")
 	(net 165 "Net-(LED56-DIN)")
@@
 	(net 189 "Net-(LED80-DIN)")
 	(net 190 "Net-(LED82-DIN)")
-	(net 191 "unconnected-(LED82-DOUT-Pad2)")
+	(net 191 "Net-(LED56-DOUT)")
 	(net 192 "Net-(LED83-DIN)")
 	(net 193 "Net-(LED84-DIN)")
@@
 			(layer "Eco2.User")
 		)
+		(fp_rect
+			(start -15 -4.7625)
+			(end -9 4.7375)
+			(stroke
+				(width 0.05)
+				(type solid)
+			)
+			(fill no)
+			(layer "Edge.Cuts")
+		)
+		(fp_rect
+			(start 9 -4.75)
+			(end 15 4.75)
+			(stroke
+				(width 0.05)
+				(type solid)
+			)
+			(fill no)
+			(layer "Edge.Cuts")
+		)
 		(fp_line
 			(start -9.045 3.4)
@@
 	(footprint "Diode_THT:D_DO-35_SOD27_P7.62mm_Horizontal"
 		(layer "F.Cu")
-		(at 285.75 59.055 -90)
+		(at 277.415625 59.055 -90)
 		(descr "Diode, DO-35_SOD27 series, Axial, Horizontal, pin pitch=7.62mm, , length*diameter=4*2mm^2, , http://www.diodes.com/_files/packages/DO-35.pdf")
 		(tags "Diode DO-35_SOD27 series Axial Horizontal pin pitch 7.62mm  length 4mm diameter 2mm")
@@
 			(layer "Eco2.User")
 		)
+		(fp_rect
+			(start -4.75 -15)
+			(end 4.75 -9)
+			(stroke
+				(width 0.05)
+				(type solid)
+			)
+			(fill no)
+			(layer "Edge.Cuts")
+		)
+		(fp_rect
+			(start -4.75 9)
+			(end 4.75 15)
+			(stroke
+				(width 0.05)
+				(type solid)
+			)
+			(fill no)
+			(layer "Edge.Cuts")
+		)
 		(fp_line
 			(start -9.045 3.4)
@@
 			(layer "Eco2.User")
 		)
+		(fp_rect
+			(start -15 -4.75)
+			(end -9 4.75)
+			(stroke
+				(width 0.05)
+				(type solid)
+			)
+			(fill no)
+			(layer "Edge.Cuts")
+		)
+		(fp_rect
+			(start 9 -4.75)
+			(end 15 4.75)
+			(stroke
+				(width 0.05)
+				(type solid)
+			)
+			(fill no)
+			(layer "Edge.Cuts")
+		)
 		(fp_line
 			(start -9.045 3.4)
@@
 	(footprint "Diode_THT:D_DO-35_SOD27_P7.62mm_Horizontal"
 		(layer "F.Cu")
-		(at 278.60625 116.205 -90)
+		(at 270.271875 116.205 -90)
 		(descr "Diode, DO-35_SOD27 series, Axial, Horizontal, pin pitch=7.62mm, , length*diameter=4*2mm^2, , http://www.diodes.com/_files/packages/DO-35.pdf")
 		(tags "Diode DO-35_SOD27 series Axial Horizontal pin pitch 7.62mm  length 4mm diameter 2mm")
@@
 			(layer "Eco2.User")
 		)
+		(fp_rect
+			(start -53 -4.75)
+			(end -47 4.75)
+			(stroke
+				(width 0.05)
+				(type solid)
+			)
+			(fill no)
+			(layer "Edge.Cuts")
+		)
+		(fp_rect
+			(start 47 -4.75)
+			(end 53 4.75)
+			(stroke
+				(width 0.05)
+				(type solid)
+			)
+			(fill no)
+			(layer "Edge.Cuts")
+		)
 		(fp_line
 			(start -9.045 3.4)
@@
 			(layers "B.Cu" "B.Mask" "B.Paste")
 			(roundrect_rratio 0.1)
-			(net 113 "Net-(LED5-DIN)")
+			(net 113 "Net-(LED6-DOUT)")
 			(pinfunction "DOUT")
 			(pintype "output")
@@
 			(layers "B.Cu" "B.Mask" "B.Paste")
 			(roundrect_rratio 0.1)
-			(net 114 "Net-(LED6-DIN)")
+			(net 112 "Net-(LED5-DOUT)")
 			(pinfunction "DIN")
 			(pintype "input")
@@
 			(layers "B.Cu" "B.Mask" "B.Paste")
 			(roundrect_rratio 0.1)
-			(net 107 "Net-(LED1-DOUT)")
+			(net 116 "Net-(LED18-DIN)")
 			(pinfunction "DIN")
 			(pintype "input")
@@
 			(layers "B.Cu" "B.Mask" "B.Paste")
 			(roundrect_rratio 0.1)
-			(net 109 "Net-(LED1-DIN)")
+			(net 109 "Net-(LED2-DOUT)")
 			(pinfunction "DOUT")
 			(pintype "output")
@@
 			(layers "B.Cu" "B.Mask" "B.Paste")
 			(roundrect_rratio 0.1)
-			(net 110 "Net-(LED2-DIN)")
+			(net 107 "Net-(LED1-DOUT)")
 			(pinfunction "DIN")
 			(pintype "input")
@@
 			(layers "B.Cu" "B.Mask" "B.Paste")
 			(roundrect_rratio 0.1)
-			(net 111 "Net-(LED3-DIN)")
+			(net 111 "Net-(LED4-DOUT)")
 			(pinfunction "DOUT")
 			(pintype "output")
@@
 			(layers "B.Cu" "B.Mask" "B.Paste")
 			(roundrect_rratio 0.1)
-			(net 112 "Net-(LED4-DIN)")
+			(net 110 "Net-(LED3-DOUT)")
 			(pinfunction "DIN")
 			(pintype "input")
@@
 			(layers "B.Cu" "B.Mask" "B.Paste")
 			(roundrect_rratio 0.1)
-			(net 191 "unconnected-(LED82-DOUT-Pad2)")
+			(net 164 "Net-(LED55-DIN)")
 			(pinfunction "DOUT")
-			(pintype "output+no_connect")
+			(pintype "output")
 		)
 		(pad "3" smd roundrect
@@
 			(layers "B.Cu" "B.Mask" "B.Paste")
 			(roundrect_rratio 0.1)
-			(net 109 "Net-(LED1-DIN)")
+			(net 117 "/LEDs/DIN")
 			(pinfunction "DIN")
 			(pintype "input")
@@
 			(layers "B.Cu" "B.Mask" "B.Paste")
 			(roundrect_rratio 0.1)
-			(net 114 "Net-(LED6-DIN)")
+			(net 114 "Net-(LED7-DOUT)")
 			(pinfunction "DOUT")
 			(pintype "output")
@@
 			(layers "B.Cu" "B.Mask" "B.Paste")
 			(roundrect_rratio 0.1)
-			(net 115 "Net-(LED7-DIN)")
+			(net 113 "Net-(LED6-DOUT)")
 			(pinfunction "DIN")
 			(pintype "input")
@@
 			(layers "B.Cu" "B.Mask" "B.Paste")
 			(roundrect_rratio 0.1)
-			(net 112 "Net-(LED4-DIN)")
+			(net 112 "Net-(LED5-DOUT)")
 			(pinfunction "DOUT")
 			(pintype "output")
@@
 			(layers "B.Cu" "B.Mask" "B.Paste")
 			(roundrect_rratio 0.1)
-			(net 113 "Net-(LED5-DIN)")
+			(net 111 "Net-(LED4-DOUT)")
 			(pinfunction "DIN")
 			(pintype "input")
@@
 			(layers "B.Cu" "B.Mask" "B.Paste")
 			(roundrect_rratio 0.1)
-			(net 116 "Net-(LED8-DIN)")
+			(net 116 "Net-(LED18-DIN)")
 			(pinfunction "DOUT")
 			(pintype "output")
@@
 			(layers "B.Cu" "B.Mask" "B.Paste")
 			(roundrect_rratio 0.1)
-			(net 117 "/LEDs/DIN")
+			(net 115 "Net-(LED8-DOUT)")
 			(pinfunction "DIN")
 			(pintype "input")
@@
 			(layers "B.Cu" "B.Mask" "B.Paste")
 			(roundrect_rratio 0.1)
-			(net 110 "Net-(LED2-DIN)")
+			(net 110 "Net-(LED3-DOUT)")
 			(pinfunction "DOUT")
 			(pintype "output")
@@
 			(layers "B.Cu" "B.Mask" "B.Paste")
 			(roundrect_rratio 0.1)
-			(net 111 "Net-(LED3-DIN)")
+			(net 109 "Net-(LED2-DOUT)")
 			(pinfunction "DIN")
 			(pintype "input")
@@
 			(layers "B.Cu" "B.Mask" "B.Paste")
 			(roundrect_rratio 0.1)
-			(net 163 "Net-(LED55-DOUT)")
+			(net 163 "unconnected-(LED55-DOUT-Pad2)")
 			(pinfunction "DOUT")
-			(pintype "output")
+			(pintype "output+no_connect")
 		)
 		(pad "3" smd roundrect
@@
 			(layers "B.Cu" "B.Mask" "B.Paste")
 			(roundrect_rratio 0.1)
-			(net 163 "Net-(LED55-DOUT)")
+			(net 191 "Net-(LED56-DOUT)")
 			(pinfunction "DIN")
 			(pintype "input")
@@
 			(layers "B.Cu" "B.Mask" "B.Paste")
 			(roundrect_rratio 0.1)
-			(net 115 "Net-(LED7-DIN)")
+			(net 115 "Net-(LED8-DOUT)")
 			(pinfunction "DOUT")
 			(pintype "output")
@@
 			(layers "B.Cu" "B.Mask" "B.Paste")
 			(roundrect_rratio 0.1)
-			(net 116 "Net-(LED8-DIN)")
+			(net 114 "Net-(LED7-DOUT)")
 			(pinfunction "DIN")
 			(pintype "input")
@@
 			(layers "B.Cu" "B.Mask" "B.Paste")
 			(roundrect_rratio 0.1)
-			(net 164 "Net-(LED55-DIN)")
+			(net 191 "Net-(LED56-DOUT)")
 			(pinfunction "DOUT")
 			(pintype "output")
@@
 	)
 	(segment
-		(start 298.73875 110.525)
-		(end 286.8325 110.525)
-		(width 0.2)
-		(layer "B.Cu")
-		(net 67)
-	)
-	(segment
 		(start 272.545 43.85)
 		(end 272.545 72.425)
@@
 	)
 	(segment
+		(start 286.8325 110.525)
+		(end 295.4565 101.901)
+		(width 0.2)
+		(layer "B.Cu")
+		(net 67)
+	)
+	(segment
 		(start 293.97625 129.575)
 		(end 293.97625 117.66875)
@@
 	)
 	(segment
+		(start 295.4565 101.901)
+		(end 304.11775 101.901)
+		(width 0.2)
+		(layer "B.Cu")
+		(net 67)
+	)
+	(segment
 		(start 267.7825 120.05)
 		(end 258.2575 129.575)
@@
 	)
 	(segment
-		(start 308.26375 101)
-		(end 298.73875 110.525)
+		(start 272.545 72.425)
+		(end 282.07 81.95)
 		(width 0.2)
 		(layer "B.Cu")
@@
 	)
 	(segment
-		(start 272.545 72.425)
-		(end 282.07 81.95)
+		(start 304.11775 101.901)
+		(end 305.01875 101)
 		(width 0.2)
 		(layer "B.Cu")
@@
 	)
 	(segment
+		(start 286.376875 72.628125)
+		(end 279.796875 72.628125)
+		(width 0.2)
+		(layer "B.Cu")
+		(net 75)
+	)
+	(segment
 		(start 287.63 71.375)
-		(end 287.63 68.555)
-		(width 0.175)
+		(end 286.376875 72.628125)
+		(width 0.2)
 		(layer "B.Cu")
 		(net 75)
 	)
 	(segment
-		(start 287.63 68.555)
-		(end 285.75 66.675)
-		(width 0.175)
+		(start 277.415625 70.246875)
+		(end 277.415625 66.675)
+		(width 0.2)
+		(layer "B.Cu")
+		(net 75)
+	)
+	(segment
+		(start 279.796875 72.628125)
+		(end 277.415625 70.246875)
+		(width 0.2)
 		(layer "B.Cu")
 		(net 75)
@@
 	)
 	(segment
-		(start 280.48625 125.705)
-		(end 278.60625 123.825)
-		(width 0.175)
+		(start 272.882308 129.176)
+		(end 279.83525 129.176)
+		(width 0.2)
 		(layer "B.Cu")
 		(net 77)
 	)
 	(segment
-		(start 280.48625 128.525)
-		(end 280.48625 125.705)
-		(width 0.175)
+		(start 270.271875 123.825)
+		(end 270.271875 126.565567)
+		(width 0.2)
+		(layer "B.Cu")
+		(net 77)
+	)
+	(segment
+		(start 270.271875 126.565567)
+		(end 272.882308 129.176)
+		(width 0.2)
+		(layer "B.Cu")
+		(net 77)
+	)
+	(segment
+		(start 279.83525 129.176)
+		(end 280.48625 128.525)
+		(width 0.2)
 		(layer "B.Cu")
 		(net 77)
@@
 	)
 	(segment
-		(start 310.645 72.52)
+		(start 311.94375 45.14875)
 		(end 311.94375 73.81875)
 		(width 0.2)
@@
 	)
 	(segment
-		(start 310.645 43.85)
-		(end 310.645 72.52)
-		(width 0.2)
-		(layer "B.Cu")
-		(net 79)
-	)
-	(segment
 		(start 311.94375 144.945)
 		(end 311.94375 96.440625)
@@
 		(width 0.2)
 		(layer "B.Cu")
+		(net 79)
+	)
+	(segment
+		(start 310.645 43.85)
+		(end 311.94375 45.14875)
+		(width 0.2)
+		(layer "B.Cu")
