File: pcb/LowJungle.kicad_pcb (KiCad board)
At the start: 2 copper layers, 378.6 x 152.4 mm, 255 parts

Commit message: Finished schematic
Other:
- board size 378.6 x 152.4 mm -> 371.5 x 133.3 mm
Changed lines of the file:
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@@
 	)
 	(gr_rect
-		(start 21.43125 21.43125)
-		(end 400.05 173.83125)
+		(start 19.048125 23.8175)
+		(end 390.526875 157.1625)
 		(stroke
 			(width 0.05)

Commit message: Started routing
Parts:
- added C1: 10uF, Capacitor_SMD:C_0805_2012Metric_Pad1.18x1.45mm_HandSolder, F.Cu at (23.4, 33.2)
- added C10: 100nF, Capacitor_SMD:C_0805_2012Metric_Pad1.18x1.45mm_HandSolder, B.Cu at (369.1, 36.8)
- added C11: 100nF, Capacitor_SMD:C_0805_2012Metric_Pad1.18x1.45mm_HandSolder, B.Cu at (378.6, 32.1)
- added C12: 10uF, Capacitor_SMD:C_0805_2012Metric_Pad1.18x1.45mm_HandSolder, B.Cu at (325.7, 26.3)
- added C13: 10uF, Capacitor_SMD:C_0805_2012Metric_Pad1.18x1.45mm_HandSolder, B.Cu at (333.4, 26.3)
- added C14: 10uF, Capacitor_SMD:C_0805_2012Metric_Pad1.18x1.45mm_HandSolder, B.Cu at (329.6, 26.3)
- added C15: 1uF, Capacitor_SMD:C_0805_2012Metric_Pad1.18x1.45mm_HandSolder, F.Cu at (370.6, 48.9)
- added C16: 1uF, Capacitor_SMD:C_0805_2012Metric_Pad1.18x1.45mm_HandSolder, F.Cu at (370.6, 52.8)
- added C2: 10uF, Capacitor_SMD:C_0805_2012Metric_Pad1.18x1.45mm_HandSolder, F.Cu at (23.4, 59.0)
- added C3: 10uF, Capacitor_SMD:C_0805_2012Metric_Pad1.18x1.45mm_HandSolder, F.Cu at (23.4, 80.8)
- added C4: 10uF, Capacitor_SMD:C_0805_2012Metric_Pad1.18x1.45mm_HandSolder, F.Cu at (23.4, 99.8)
- added C5: 10uF, Capacitor_SMD:C_0805_2012Metric_Pad1.18x1.45mm_HandSolder, F.Cu at (23.4, 118.4)
- added C6: 10uF, Capacitor_SMD:C_0805_2012Metric_Pad1.18x1.45mm_HandSolder, F.Cu at (23.4, 136.8)
- added C7: 100nF, Capacitor_SMD:C_0805_2012Metric_Pad1.18x1.45mm_HandSolder, B.Cu at (366.7, 32.0)
- added C8: 10uF, Capacitor_SMD:C_0805_2012Metric_Pad1.18x1.45mm_HandSolder, B.Cu at (369.1, 32.0)
- added C9: 1uF, Capacitor_SMD:C_0805_2012Metric_Pad1.18x1.45mm_HandSolder, B.Cu at (364.3, 36.8)
- added H1: MountingHole_Pad, MountingHole:MountingHole_3.2mm_M3_DIN965_Pad_TopOnly, F.Cu at (22.6, 27.4)
- added H2: MountingHole_Pad, MountingHole:MountingHole_3.2mm_M3_DIN965_Pad_TopOnly, F.Cu at (146.4, 27.4)
- added H3: MountingHole_Pad, MountingHole:MountingHole_3.2mm_M3_DIN965_Pad_TopOnly, F.Cu at (319.1, 90.5)
- added H4: MountingHole_Pad, MountingHole:MountingHole_3.2mm_M3_DIN965_Pad_TopOnly, F.Cu at (22.6, 153.6)
- added H5: MountingHole_Pad, MountingHole:MountingHole_3.2mm_M3_DIN965_Pad_TopOnly, F.Cu at (387.0, 27.4)
- added H6: MountingHole_Pad, MountingHole:MountingHole_3.2mm_M3_DIN965_Pad_TopOnly, F.Cu at (145.3, 153.6)
- added H7: MountingHole_Pad, MountingHole:MountingHole_3.2mm_M3_DIN965_Pad_TopOnly, F.Cu at (387.0, 153.6)
- added J1: JTAG, Connector_PinHeader_1.00mm:PinHeader_1x04_P1.00mm_Vertical, F.Cu at (338.6, 39.6)
- added J2: 3.3V, Connector_PinHeader_1.00mm:PinHeader_1x02_P1.00mm_Vertical, F.Cu at (373.3, 48.7)
- added J3: 5V, Connector_PinHeader_1.00mm:PinHeader_1x02_P1.00mm_Vertical, F.Cu at (373.3, 52.9)
- added JP1: Backlight_OUT, Jumper:SolderJumper-2_P1.3mm_Bridged2Bar_RoundedPad1.0x1.5mm, F.Cu at (297.9, 49.6)
- added JP2: Backlight_VBUS, Jumper:SolderJumper-2_P1.3mm_Bridged2Bar_RoundedPad1.0x1.5mm, F.Cu at (312.3, 49.1)
- added LDO1: ME6211C33M5G-N, easyeda2kicad:SOT-23-5_L3.0-W1.7-P0.95-LS2.8-BL, F.Cu at (365.4, 50.8)
- added LED86: KS33_SK6812MINI-E, PCM_marbastlib-xp-gateron_lp:LED_KS33_6028R, B.Cu at (329.8, 41.7)
- added LED87: KS33_SK6812MINI-E, PCM_marbastlib-xp-gateron_lp:LED_KS33_6028R, B.Cu at (329.8, 36.9)
- added LED88: KS33_SK6812MINI-E, PCM_marbastlib-xp-gateron_lp:LED_KS33_6028R, B.Cu at (329.8, 32.1)
- added LED89: KS33_SK6812MINI-E, PCM_marbastlib-xp-gateron_lp:LED_KS33_6028R, B.Cu at (336.6, 105.5)
- added LED90: KS33_SK6812MINI-E, PCM_marbastlib-xp-gateron_lp:LED_KS33_6028R, B.Cu at (343.1, 105.5)
- added LED91: KS33_SK6812MINI-E, PCM_marbastlib-xp-gateron_lp:LED_KS33_6028R, B.Cu at (349.4, 105.5)
- added LED92: KS33_SK6812MINI-E, PCM_marbastlib-xp-gateron_lp:LED_KS33_6028R, B.Cu at (355.9, 105.5)
- added LED93: KS33_SK6812MINI-E, PCM_marbastlib-xp-gateron_lp:LED_KS33_6028R, B.Cu at (362.2, 105.4)
- added LED94: KS33_SK6812MINI-E, PCM_marbastlib-xp-gateron_lp:LED_KS33_6028R, B.Cu at (368.6, 105.4)
- added Q1: CJ2301 S1, easyeda2kicad:SOT-23-3_L3.0-W1.7-P0.95-LS2.9-BR, F.Cu at (304.1, 49.7)
- added Q2: SI2302_C2891732, easyeda2kicad:SOT-23-3_L2.9-W1.3-P1.90-LS2.4-BR, F.Cu at (304.1, 53.5)
- added R1: 10k, Resistor_SMD:R_0805_2012Metric_Pad1.20x1.40mm_HandSolder, B.Cu at (364.3, 32.0)
- added R2: 10k, Resistor_SMD:R_0805_2012Metric_Pad1.20x1.40mm_HandSolder, B.Cu at (382.1, 32.1)
- added R3: 5.1k, Resistor_SMD:R_0805_2012Metric_Pad1.20x1.40mm_HandSolder, B.Cu at (310.8, 27.4)
- added R4: 5.1k, Resistor_SMD:R_0805_2012Metric_Pad1.20x1.40mm_HandSolder, B.Cu at (307.7, 27.4)
- added R5: 10k, Resistor_SMD:R_0805_2012Metric_Pad1.20x1.40mm_HandSolder, F.Cu at (308.3, 52.2)
- added R6: 5.1k, Resistor_SMD:R_0805_2012Metric_Pad1.20x1.40mm_HandSolder, F.Cu at (298.5, 53.4)
- added SW1: RotaryEncoder_Switch, Rotary_Encoder:RotaryEncoder_Alps_EC11E-Switch_Vertical_H20mm_CircularMountingHoles, F.Cu at (381.2, 40.6)
- added SW2: GT-TC029A-H020-L1N, easyeda2kicad:SW-SMD_L3.9-W2.9-LS5.0, B.Cu at (368.4, 27.4)
- added SW3: GT-TC029A-H020-L1N, easyeda2kicad:SW-SMD_L3.9-W2.9-LS5.0, B.Cu at (376.8, 27.4)
- added TP1: RX, TestPoint:TestPoint_Pad_D1.0mm, B.Cu at (338.6, 37.4)
- added TP2: TX, TestPoint:TestPoint_Pad_D1.0mm, B.Cu at (338.6, 35.2)
- added U1: ESP32-S3-WROOM-1(N8R2), easyeda2kicad:WIRELM-SMD_ESP32-S3-WROOM-1, B.Cu at (350.0, 41.5)
- added U2: GT-USB-7010ASV, easyeda2kicad:USB-C-SMD_G-SWITCH_GT-USB-7010ASV, F.Cu at (319.1, 28.5)
- added U3: SL2.1A, easyeda2kicad:SOP-16_L10.0-W3.9-P1.27-LS6.0-BL, B.Cu at (319.6, 42.9)
- added USB1: KH-AF90DIP-112, easyeda2kicad:USB-A-TH_USB-A-F-90, B.Cu at (56.3, 34.4)
- added USB2: KH-AF90DIP-112, easyeda2kicad:USB-A-TH_USB-A-F-90, B.Cu at (379.9, 106.0)
- added USB3: DNP, easyeda2kicad:USB-A-TH_USB-A-F-90, B.Cu at (379.9, 126.2)
Connections:
- net VBUS renamed Vdrive
- D32 pad 1: unconnected-(D32-K-Pad1) -> /KeyMatrix/ROW_2
- LED1 pad 3: /LEDs/DIN -> Net-(LED1-DIN)
- LED15 pad 2: Net-(LED14-DIN) -> Net-(LED15-DOUT)
- LED15 pad 3: Net-(LED15-DIN) -> /LEDs/DIN
- LED16 pad 2: Net-(LED15-DIN) -> Net-(LED16-DOUT)
- LED16 pad 3: Net-(LED16-DIN) -> Net-(LED15-DOUT)
- LED17 pad 2: Net-(LED16-DIN) -> Net-(LED17-DOUT)
- LED17 pad 3: Net-(LED17-DIN) -> Net-(LED16-DOUT)
- LED18 pad 2: Net-(LED17-DIN) -> Net-(LED1-DIN)
- LED18 pad 3: Net-(LED18-DIN) -> Net-(LED17-DOUT)
- LED9 pad 2: Net-(LED18-DIN) -> Net-(LED14-DIN)
Routing:
- net Vdrive: track 0.00 -> 3076.2 mm, vias 0 -> 93
- net Net-(LED33-DIN): track 0.00 -> 374.4 mm, vias 0 -> 2
- net Net-(LED52-DIN): track 0.00 -> 367.2 mm, vias 0 -> 4
- net Net-(LED78-DIN): track 0.00 -> 363.4 mm, vias 0 -> 4
- net /LEDs/DIN: track 0.00 -> 322.1 mm, vias 0 -> 2
- net Net-(LED14-DIN): track 0.00 -> 312.1 mm, vias 0 -> 2
- net Net-(U3-DM3): track 0.00 -> 290.9 mm, vias 0 -> 6
- net Net-(U3-DP3): track 0.00 -> 285.7 mm, vias 0 -> 4
- net Net-(LED57-DIN): track 0.00 -> 272.8 mm, vias 0 -> 2
- net VBUS: track 0.00 -> 245.0 mm, vias 0 -> 10
- net Net-(U3-DM1): track 0.00 -> 146.1 mm, vias 0 -> 1
- net Net-(U3-DP1): track 0.00 -> 144.7 mm, vias 0 -> 1
- net Net-(U3-DP2): track 0.00 -> 121.0 mm, vias 0 -> 2
- net /KeyMatrix/COLUM_8: track 306.4 -> 191.8 mm, vias 2 -> 6
- net Net-(U3-DM2): track 0.00 -> 113.3 mm, vias 0 -> 2
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Other:
- board size 371.5 x 133.3 mm -> 371.5 x 133.4 mm
