File: pcb/key_matrix.kicad_sch (KiCad schematic)
At the start: 170 parts

Commit message: Started routing
Connections:
- net ROW_2: now also D32.1 (K)
Changed lines of the file:
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@@
+	)
+	(junction
+		(at 88.9 46.99)
+		(diameter 0)
+		(color 0 0 0 0)
 	)
 	(junction
@@
 	(wire
 		(pts
-			(xy 71.12 46.99) (xy 107.95 46.99)
+			(xy 71.12 46.99) (xy 88.9 46.99)
 		)
 		(stroke
@@
 	(wire
 		(pts
+			(xy 88.9 46.99) (xy 107.95 46.99)
+		)
+		(stroke
+			(width 0)
+			(type default)
+		)
+	)
+	(wire
+		(pts
 			(xy 113.03 113.03) (xy 113.03 127)
 		)
@@
 		)
 		(stroke
+			(width 0)
+			(type default)
+		)
+	)
+	(wire
+		(pts
+			(xy 88.9 44.45) (xy 88.9 46.99)
+		)
+		(stroke
