File: pcb/leds.kicad_sch (KiCad schematic)
At the start: 85 parts

Commit message: ledsssssss
Connections:
- net DIN: now also LED1.3 (DIN); no longer LED9.3 (DIN)
- net at LED6.2 (DOUT): now also LED7.3 (DIN); no longer LED5.3 (DIN)
- net at LED6.3 (DIN): now also LED5.2 (DOUT); no longer LED7.2 (DOUT)
- net at LED55.2 (DOUT): no longer LED72.3 (DIN)
- net at LED55.3 (DIN): now also LED82.2 (DOUT); no longer LED56.2 (DOUT)
- net at LED1.2 (DOUT): now also LED2.3 (DIN); no longer LED18.3 (DIN)
- net at LED2.2 (DOUT): now also LED3.3 (DIN); no longer LED1.3 (DIN)
- net at LED4.3 (DIN): now also LED3.2 (DOUT); no longer LED5.2 (DOUT)
- net at LED4.2 (DOUT): now also LED5.3 (DIN); no longer LED3.3 (DIN)
- net at LED8.2 (DOUT): now also LED9.3 (DIN); no longer LED7.3 (DIN)
- net at LED9.2 (DOUT): now also LED18.3 (DIN); no longer LED8.3 (DIN)
- new net: LED56.2 (DOUT), LED72.3 (DIN)
- new net: LED7.2 (DOUT), LED8.3 (DIN)

Commit message: Finished schematic
Parts:
- added C1, C2, C3, C4, C5, C6: 10uF, Capacitor_SMD:C_0805_2012Metric_Pad1.18x1.45mm_HandSolder, symbol Device:C_Small
Connections:
- net GND: now also C1.2, C2.2, C3.2, C4.2, C5.2, C6.2
- net VBUS renamed Vdrive
- net Vdrive: now also C1.1, C2.1, C3.1, C4.1, C5.1, C6.1

Commit message: Started routing
Connections:
- net DIN: now also LED15.3 (DIN); no longer LED1.3 (DIN)
- net at LED16.2 (DOUT): now also LED17.3 (DIN); no longer LED15.3 (DIN)
- net at LED16.3 (DIN): now also LED15.2 (DOUT); no longer LED17.2 (DOUT)
- net at LED18.2 (DOUT): now also LED1.3 (DIN); no longer LED17.3 (DIN)
- net at LED18.3 (DIN): now also LED17.2 (DOUT); no longer LED9.2 (DOUT)
- net at LED14.3 (DIN): now also LED9.2 (DOUT); no longer LED15.2 (DOUT)
