File: pcb/usb.kicad_sch (KiCad schematic)
At the start: 19 parts, among them Q1 CJ2301 S1, Q2 SI2302_C2891732, U2 GT-USB-7010ASV, U3 SL2.1A

Commit message: Started routing
Connections:
- net GND: now also USB1.4 (GND), USB2.4 (GND), USB3.4 (GND)
- net VBUS: now also USB2.1 (VCC), USB3.1 (VCC)
- net Vdrive: now also USB1.1 (VCC)
